File: carte driver/carte driver.kicad_pcb (KiCad board)
At the start: 2 copper layers, 120 x 50 mm, 38 parts, among them J1 UART CP, J10 STEPPER 4, J11 STEPPER 3, J2 Conn_01x03, J3 UART BONUS, J6 STEPPER G, J7 STEPPER D, J8 STEPPER 1, J9 STEPPER 2, SW2 SW_DIP_x02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

Commit message: c'est l'heure de dodo j'ai bien taffé
Parts:
- added D2: LED_Small, LED_SMD:LED_1206_3216Metric, B.Cu at (143.0, 143.0)
- added J4: Conn_01x02, Connector_Molex:Molex_KK-254_AE-6410-02A_1x02_P2.54mm_Vertical, F.Cu at (140.0, 138.5)
- added R1: 1k, Resistor_SMD:R_1206_3216Metric_Pad1.30x1.75mm_HandSolder, F.Cu at (130.5, 138.0)
- added R2: 1k, Resistor_SMD:R_1206_3216Metric_Pad1.30x1.75mm_HandSolder, F.Cu at (130.5, 135.5)
- added R5: 1k, Resistor_SMD:R_1206_3216Metric_Pad1.30x1.75mm_HandSolder, B.Cu at (140.7, 143.0)
- D3, R3: moved to B.Cu
- moved R3 116.3 mm to (29.5, 157.0), turned to 180 degrees
- moved R4 115.2 mm to (29.5, 157.0), turned to 180 degrees
- moved D3 111.9 mm to (29.5, 159.5), turned to 180 degrees
- moved D4 110.6 mm to (29.5, 159.5), turned to 180 degrees
- moved J2 96.5 mm to (29.2, 152.5), turned to 90 degrees
- moved C5 64.4 mm to (127.0, 166.6), turned to -90 degrees
- moved D1 34.1 mm to (143.1, 162.5), turned to 180 degrees
- moved J3 8.02 mm to (132.0, 132.5)
- moved J1 7.23 mm to (124.5, 132.5)
Connections:
- J2 pad 1: +24V -> +3.3V
- J2 pad 2: +5V -> +24V
- U10 pad 1: STEP 1 -> STEP 3
- U10 pad 12: +3.3V -> unconnected-(U10-VCC_3V3-Pad12)
- U10 pad 15: STEP 5 -> DIR 5
- U10 pad 16: DIR 5 -> STEP 5
- U10 pad 18: RX B -> unconnected-(U10-GPIO41_PDM_DATA/RX1-Pad18)
- U10 pad 19: TX B -> Net-(U10-GPIO42_PDM_CLK/TX1)
- U10 pad 2: DIR 1 -> DIR 3
- U10 pad 20: unconnected-(U10-GPIO10_XMCLK/ADC_BAT-Pad20) -> Net-(U10-GPIO10_XMCLK/ADC_BAT)
- U10 pad 3: STEP 2 -> STEP 1
- U10 pad 4: DIR 2 -> DIR 1
- U10 pad 5: STEP 3 -> STEP 2
- U10 pad 6: DIR 3 -> DIR 2
Routing:
- net +24V: track 0.00 -> 249.1 mm
- net +3.3V: track 0.00 -> 220.9 mm
- net EN M: track 0.00 -> 121.6 mm
- net EN: track 0.00 -> 103.4 mm, vias 0 -> 1
- net STEP 1: track 0.00 -> 91.6 mm
- net DIR 1: track 0.00 -> 90.9 mm
- net STEP 3: track 0.00 -> 84.2 mm, vias 0 -> 1
- net DIR 3: track 0.00 -> 80.7 mm, vias 0 -> 1
- net STEP 2: track 0.00 -> 58.0 mm
- net DIR 2: track 0.00 -> 57.3 mm
- net DIR 4: track 0.00 -> 43.2 mm, vias 0 -> 1
- net +5V: track 0.00 -> 43.1 mm
- net STEP 4: track 0.00 -> 41.4 mm, vias 0 -> 1
- net RX: track 0.00 -> 28.6 mm
- net DIR 5: track 0.00 -> 24.1 mm
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- added copper zone on B.Cu, net GND
- added copper zone on F.Cu, net GND

Commit message: fix
Routing:
- net DIR 6: track 8.37 -> 10.2 mm
- net STEP 6: track 9.65 -> 10.8 mm
- net +3.3V: track 220.9 -> 219.9 mm
