File: carte driver/carte driver.kicad_pcb (KiCad board)
At the start: 2 copper layers, 120 x 50 mm, 43 parts, among them J1 UART CP, J10 STEPPER 4, J11 STEPPER 3, J2 Conn_01x03, J3 UART BONUS, J4 Conn_01x02, J6 STEPPER G, J7 STEPPER D, J8 STEPPER 1, J9 STEPPER 2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

Commit message: debut etiquettes
Parts:
- added kibuzzard-67ED8648: G***, kibuzzard-67ED8648, B.Cu at (138.1, 155.6)
- added kibuzzard-67EE6BB1: G***, kibuzzard-67EE6BB1, F.Cu at (50.4, 137.4)
- added kibuzzard-67EE6BB1: G***, kibuzzard-67EE6BB1, F.Cu at (78.6, 163.1)
- added kibuzzard-67EE6BB1: G***, kibuzzard-67EE6BB1, F.Cu at (107.2, 137.5)
- added kibuzzard-67EE6BB1: G***, kibuzzard-67EE6BB1, F.Cu at (78.9, 137.5)
- added kibuzzard-67EE6BB1: G***, kibuzzard-67EE6BB1, F.Cu at (106.9, 163.1)
- added kibuzzard-67EE6BB1: G***, kibuzzard-67EE6BB1, F.Cu at (50.4, 163.0)
- added kibuzzard-68F7E1A4: G***, kibuzzard-68F7E1A4, F.Cu at (36.9, 142.4)
- added kibuzzard-68F7E205: G***, kibuzzard-68F7E205, F.Cu at (36.8, 168.2)
- added kibuzzard-68F7E48E: G***, kibuzzard-68F7E48E, F.Cu at (65.2, 142.4)
- added kibuzzard-68F7E494: G***, kibuzzard-68F7E494, F.Cu at (65.1, 168.2)
- added kibuzzard-68F7E49A: G***, kibuzzard-68F7E49A, F.Cu at (93.9, 142.3)
- added kibuzzard-68F7E4A0: G***, kibuzzard-68F7E4A0, F.Cu at (94.2, 168.1)
- added kibuzzard-68F7E57E: G***, kibuzzard-68F7E57E, B.Cu at (136.8, 143.1)
- added kibuzzard-68F7E5B2: G***, kibuzzard-68F7E5B2, B.Cu at (135.6, 145.2)
- added kibuzzard-68F7E5C0: G***, kibuzzard-68F7E5C0, B.Cu at (138.1, 145.2)
- added kibuzzard-68F7E5C7: G***, kibuzzard-68F7E5C7, B.Cu at (133.0, 145.2)
- added kibuzzard-68F7E5D0: G***, kibuzzard-68F7E5D0, B.Cu at (130.5, 145.2)
- added kibuzzard-68F7E5E0: G***, kibuzzard-68F7E5E0, B.Cu at (127.9, 145.2)
- added kibuzzard-68F7E5E6: G***, kibuzzard-68F7E5E6, B.Cu at (125.4, 145.2)
- added kibuzzard-68F7E5EE: G***, kibuzzard-68F7E5EE, B.Cu at (122.9, 144.0)
- added kibuzzard-68F7E6E6: G***, kibuzzard-68F7E6E6, B.Cu at (134.3, 143.1)
- added kibuzzard-68F7E6FB: G***, kibuzzard-68F7E6FB, B.Cu at (135.6, 155.6)
- added kibuzzard-68F7E70E: G***, kibuzzard-68F7E70E, B.Cu at (130.5, 154.2)
- added kibuzzard-68F7E71B: G***, kibuzzard-68F7E71B, B.Cu at (129.2, 157.5)
- added kibuzzard-68F7E74E: G***, kibuzzard-68F7E74E, B.Cu at (127.9, 154.9)
- added kibuzzard-68F7E766: G***, kibuzzard-68F7E766, B.Cu at (125.4, 154.7)
- added kibuzzard-68F7E774: G***, kibuzzard-68F7E774, B.Cu at (122.9, 155.8)
- added kibuzzard-68F7E782: G***, kibuzzard-68F7E782, B.Cu at (124.1, 156.9)
- added kibuzzard-68F7E793: G***, kibuzzard-68F7E793, B.Cu at (126.7, 156.7)
- moved C6 1.03 mm to (97.6, 159.3)
- moved J8 0.76 mm to (68.8, 138.6)
- moved J10 0.75 mm to (97.9, 164.3)
- moved J11 0.58 mm to (97.5, 138.5)
- moved U6 0.52 mm to (111.8, 163.1)
- moved SW6 0.52 mm to (113.0, 159.3)
- moved J7 0.31 mm to (40.5, 164.4)
- moved C7 0.20 mm to (97.8, 133.9)
Routing:
- net +3.3V: track 219.9 -> 216.4 mm
- net EN M: track 121.6 -> 120.1 mm
- net DIR 6: track 10.2 -> 9.06 mm
- net Net-(J9-Pin_2): track 8.33 -> 8.96 mm
- net Net-(J9-Pin_4): track 9.38 -> 9.98 mm
- net Net-(J9-Pin_1): track 8.34 -> 8.93 mm
- net STEP 6: track 10.8 -> 11.3 mm

Commit message: apdavph
Parts:
- added kibuzzard-68F7E6E6: G***, kibuzzard-68F7E6E6, B.Cu at (126.7, 143.2)
Connections:
- U1 pad 3: Net-(J6-Pin_3) -> Net-(J6-Pin_1)
- U1 pad 4: Net-(J6-Pin_1) -> Net-(J6-Pin_2)
- U1 pad 5: Net-(J6-Pin_2) -> Net-(J6-Pin_3)
- U2 pad 3: Net-(J7-Pin_3) -> Net-(J7-Pin_1)
- U2 pad 4: Net-(J7-Pin_1) -> Net-(J7-Pin_2)
- U2 pad 5: Net-(J7-Pin_2) -> Net-(J7-Pin_3)
- U3 pad 3: Net-(J8-Pin_3) -> Net-(J8-Pin_1)
- U3 pad 4: Net-(J8-Pin_1) -> Net-(J8-Pin_2)
- U3 pad 5: Net-(J8-Pin_2) -> Net-(J8-Pin_3)
- U4 pad 3: Net-(J9-Pin_3) -> Net-(J9-Pin_1)
- U4 pad 4: Net-(J9-Pin_1) -> Net-(J9-Pin_2)
- U4 pad 5: Net-(J9-Pin_2) -> Net-(J9-Pin_3)
- U5 pad 3: Net-(J11-Pin_3) -> Net-(J11-Pin_1)
- U5 pad 4: Net-(J11-Pin_1) -> Net-(J11-Pin_2)
- U5 pad 5: Net-(J11-Pin_2) -> Net-(J11-Pin_3)
- U6 pad 3: Net-(J10-Pin_3) -> Net-(J10-Pin_1)
- U6 pad 4: Net-(J10-Pin_1) -> Net-(J10-Pin_2)
- U6 pad 5: Net-(J10-Pin_2) -> Net-(J10-Pin_3)
Routing:
- net Net-(J11-Pin_3): track 18.7 -> 9.74 mm
- net Net-(J9-Pin_3): track 18.7 -> 10.0 mm
- net Net-(J10-Pin_3): track 18.5 -> 9.94 mm
- net Net-(J6-Pin_3): track 18.5 -> 10.0 mm
- net Net-(J8-Pin_3): track 18.7 -> 10.3 mm
- net Net-(J7-Pin_3): track 18.4 -> 10.0 mm
- net +3.3V: track 216.4 -> 212.5 mm
- net EN M: track 120.1 -> 118.1 mm
- net EN: track 102.9 -> 100.9 mm
- net +24V: track 249.5 -> 247.7 mm
- net Net-(J6-Pin_2): track 8.33 -> 10.0 mm
- net Net-(J6-Pin_1): track 8.34 -> 10.0 mm
- net Net-(J8-Pin_2): track 8.78 -> 10.4 mm
- net Net-(J8-Pin_1): track 8.75 -> 10.3 mm
- net Net-(J7-Pin_2): track 8.83 -> 10.0 mm
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
Commit message: caph
Routing:
- net +24V: track 247.7 -> 239.0 mm
Changed lines of the file:
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@@
 			(psa4output no)
 			(plot_black_and_white yes)
+			(plotinvisibletext no)
 			(sketchpadsonfab no)
 			(plotpadnumbers no)
@@
 	)
 	(segment
-		(start 105.4025 171.99)
-		(end 104.99 171.99)
+		(start 69.5325 133.725177)
+		(end 73.33 137.522677)
 		(width 2)
 		(layer "F.Cu")
@@
 	)
 	(segment
-		(start 104.99 171.99)
-		(end 103 170)
-		(width 2)
-		(layer "F.Cu")
-		(net 1)
-	)
-	(segment
 		(start 31.05 157)
 		(end 38.517322 157)
@@
 	)
 	(segment
-		(start 103 170)
-		(end 103 154.5)
+		(start 69.25 148.75)
+		(end 72.42 148.75)
 		(width 2)
 		(layer "F.Cu")
@@
 	)
 	(segment
-		(start 40.5325 133.515178)
-		(end 45 137.982678)
+		(start 73.5 156.5)
+		(end 73.5 150.17)
 		(width 2)
 		(layer "F.Cu")
@@
 	)
 	(segment
-		(start 68.7825 159.247678)
-		(end 70.752322 159.247678)
+		(start 97.63 159.27)
+		(end 102.98 159.27)
 		(width 2)
 		(layer "F.Cu")
@@
 	)
 	(segment
-		(start 73.5 150.17)
-		(end 73.33 150)
+		(start 73.08 148.75)
+		(end 47.25 148.75)
 		(width 2)
 		(layer "F.Cu")
@@
 	)
 	(segment
-		(start 101.5 150.1475)
-		(end 101.6475 150)
-		(width 2)
-		(layer "F.Cu")
-		(net 1)
-	)
-	(segment
-		(start 73.33 150)
-		(end 101.6475 150)
+		(start 45 137.982678)
+		(end 45 149)
 		(width 2)
 		(layer "F.Cu")
@@
 	)
 	(segment
-		(start 47.25 148.75)
-		(end 46 150)
+		(start 101.5 150.1475)
+		(end 101.5 137.4)
 		(width 2)
 		(layer "F.Cu")
@@
 	)
 	(segment
-		(start 97.6 159.3)
-		(end 97.63 159.27)
+		(start 104.99 171.99)
+		(end 103 170)
 		(width 2)
 		(layer "F.Cu")
@@
 	)
 	(segment
-		(start 97.8 133.867678)
-		(end 97.967678 133.867678)
+		(start 40.7825 159.265178)
+		(end 46 159.265178)
 		(width 2)
 		(layer "F.Cu")
@@
 	)
 	(segment
-		(start 76.9325 146.3975)
-		(end 73.33 150)
+		(start 73.67 150)
+		(end 101.6475 150)
 		(width 2)
 		(layer "F.Cu")
@@
 	)
 	(segment
-		(start 73.33 137.522677)
-		(end 73.33 150)
+		(start 97.967678 133.867678)
+		(end 97.8 133.867678)
 		(width 2)
 		(layer "F.Cu")
@@
 	)
 	(segment
-		(start 70.752322 159.247678)
-		(end 73.5 156.5)
+		(start 68.7825 159.247678)
+		(end 73.5 159.247678)
 		(width 2)
 		(layer "F.Cu")
@@
 	)
 	(segment
-		(start 45 149)
+		(start 47.25 148.75)
 		(end 46 150)
 		(width 2)
@@
 	)
 	(segment
-		(start 101.5 137.4)
-		(end 101.5 150.1475)
-		(width 2)
-		(layer "F.Cu")
-		(net 1)
-	)
-	(segment
-		(start 73.5 150.17)
-		(end 72.08 148.75)
+		(start 40.5325 133.515178)
+		(end 45 137.982678)
 		(width 2)
 		(layer "F.Cu")
@@
 	)
 	(segment
-		(start 69.5325 133.725177)
-		(end 73.33 137.522677)
+		(start 44.72 150)
+		(end 29.2 150)
 		(width 2)
 		(layer "F.Cu")
@@
 	)
 	(segment
-		(start 73.5 156.5)
-		(end 73.5 150.17)
+		(start 98 133.842855)
+		(end 97.824823 133.842855)
 		(width 2)
 		(layer "F.Cu")
@@
 	)
 	(segment
-		(start 97.63 159.27)
-		(end 99.73 159.27)
+		(start 102.98 159.27)
+		(end 103 159.25)
 		(width 2)
 		(layer "F.Cu")
@@
 	)
 	(segment
-		(start 44.72 150)
-		(end 29.2 150)
+		(start 46 170.671317)
+		(end 46 154.047678)
 		(width 2)
 		(layer "F.Cu")
@@
 	)
 	(segment
-		(start 45 137.982678)
-		(end 45 149)
+		(start 97.824823 133.842855)
+		(end 97.8 133.867678)
 		(width 2)
 		(layer "F.Cu")
@@
 	)
 	(segment
-		(start 98 133.842855)
-		(end 97.824823 133.842855)
+		(start 72.42 148.75)
+		(end 73.67 150)
 		(width 2)
 		(layer "F.Cu")
@@
 	)
 	(segment
-		(start 46 170.671317)
-		(end 46 154.047678)
+		(start 73.5 169.921317)
+		(end 73.5 156.5)
 		(width 2)
 		(layer "F.Cu")
@@
 	)
 	(segment
-		(start 97.824823 133.842855)
-		(end 97.8 133.867678)
+		(start 47.366183 172.0375)
+		(end 46 170.671317)
 		(width 2)
 		(layer "F.Cu")
@@
 	)
 	(segment
-		(start 73.5 169.921317)
-		(end 73.5 156.5)
+		(start 48.4325 147.5675)
+		(end 48.4325 146.2875)
 		(width 2)
 		(layer "F.Cu")
@@
 	)
 	(segment
-		(start 47.366183 172.0375)
-		(end 46 170.671317)
+		(start 97.6 159.3)
+		(end 97.63 159.27)
 		(width 2)
 		(layer "F.Cu")
@@
 	)
 	(segment
-		(start 40.7825 159.265178)
-		(end 46 154.047678)
+		(start 103 151.6475)
+		(end 101.5 150.1475)
 		(width 2)
 		(layer "F.Cu")
@@
 	)
 	(segment
-		(start 103 156)
-		(end 103 151.6475)
+		(start 101.5 137.4)
+		(end 97.967678 133.867678)
 		(width 2)
 		(layer "F.Cu")
@@
 	)
 	(segment
-		(start 72.08 148.75)
-		(end 47.25 148.75)
+		(start 48.4325 172.0375)
+		(end 47.366183 172.0375)
 		(width 2)
 		(layer "F.Cu")
@@
 	)
 	(segment
-		(start 48.4325 172.0375)
-		(end 47.366183 172.0375)
+		(start 103 170)
+		(end 103 151.6475)
 		(width 2)
 		(layer "F.Cu")
@@
 	)
 	(segment
-		(start 48.4325 146.2875)
-		(end 44.72 150)
+		(start 44.72 150)
+		(end 46 150)
 		(width 2)
 		(layer "F.Cu")
@@
 	)
 	(segment
-		(start 44.72 150)
-		(end 46 150)
+		(start 73.33 137.522677)
+		(end 73.33 148.5)
 		(width 2)
 		(layer "F.Cu")
@@
 	)
 	(segment
-		(start 97.967678 133.867678)
-		(end 101.5 137.4)
+		(start 73.67 149.66)
+		(end 76.9325 146.3975)
 		(width 2)
 		(layer "F.Cu")
@@
 	)
 	(segment
-		(start 99.73 159.27)
-		(end 103 156)
+		(start 47.25 148.75)
+		(end 48.4325 147.5675)
 		(width 2)
 		(layer "F.Cu")
@@
 	)
 	(segment
-		(start 103 151.6475)
-		(end 101.5 150.1475)
+		(start 105.4025 171.99)
+		(end 104.99 171.99)
 		(width 2)
 		(layer "F.Cu")
