File: carte driver/_autosave-carte driver.kicad_pcb (KiCad board)
At the start: 2 copper layers, 120 x 50 mm, 74 parts, among them J1 UART CP, J10 STEPPER 4, J11 STEPPER 3, J2 Conn_01x03, J3 UART BONUS, J4 Conn_01x02, J6 STEPPER G, J7 STEPPER D, J8 STEPPER 1, J9 STEPPER 2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

Commit message: ajout logo
Parts:
- added G***: LOGO, LOGO, F.Cu at (130.7, 150.0)
- added G***: LOGO, LOGO, B.Cu at (74.8, 156.5)
Other:
- board text added: "By Oscar Yosh GRIVELET"
- board text added: "Carte_Driver_2026_V1"
