File: carte driver v2/carte driver v2.kicad_pcb (KiCad board)
At the start: 2 copper layers, 103 x 50 mm, 43 parts, among them J1 UART CP, J10 STEPPER 2, J11 STEPPER 4, J2 UART BONUS, J3 conn 24v, J4 conn 5v, J6 STEPPER G, J7 STEPPER 1, J8 STEPPER 3, J9 STEPPER D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

Commit message: deso alph
Parts:
- added G***: LOGO, LOGO, B.Cu at (124.4, 114.8)
- added kibuzzard-67ED8648: G***, kibuzzard-67ED8648, F.Cu at (166.3, 113.1)
- added kibuzzard-68F7E1A4: G***, kibuzzard-68F7E1A4, B.Cu at (81.4, 89.5)
- added kibuzzard-68F7E205: G***, kibuzzard-68F7E205, B.Cu at (81.3, 125.4)
- added kibuzzard-68F7E48E: G***, kibuzzard-68F7E48E, B.Cu at (107.9, 89.5)
- added kibuzzard-68F7E494: G***, kibuzzard-68F7E494, B.Cu at (107.8, 125.4)
- added kibuzzard-68F7E49A: G***, kibuzzard-68F7E49A, B.Cu at (134.4, 89.5)
- added kibuzzard-68F7E4A0: G***, kibuzzard-68F7E4A0, B.Cu at (134.3, 125.4)
- added kibuzzard-68F7E57E: G***, kibuzzard-68F7E57E, F.Cu at (165.0, 100.4)
- added kibuzzard-68F7E5B2: G***, kibuzzard-68F7E5B2, F.Cu at (163.8, 102.5)
- added kibuzzard-68F7E5C0: G***, kibuzzard-68F7E5C0, F.Cu at (166.3, 102.4)
- added kibuzzard-68F7E5C7: G***, kibuzzard-68F7E5C7, F.Cu at (161.2, 102.4)
- added kibuzzard-68F7E5D0: G***, kibuzzard-68F7E5D0, F.Cu at (158.8, 102.0)
- added kibuzzard-68F7E5E0: G***, kibuzzard-68F7E5E0, F.Cu at (156.2, 102.3)
- added kibuzzard-68F7E5E6: G***, kibuzzard-68F7E5E6, F.Cu at (153.7, 102.0)
- added kibuzzard-68F7E5EE: G***, kibuzzard-68F7E5EE, F.Cu at (151.2, 101.1)
- added kibuzzard-68F7E6E6: G***, kibuzzard-68F7E6E6, F.Cu at (162.6, 100.6)
- added kibuzzard-68F7E6FB: G***, kibuzzard-68F7E6FB, F.Cu at (163.8, 112.9)
- added kibuzzard-68F7E70E: G***, kibuzzard-68F7E70E, F.Cu at (158.8, 111.5)
- added kibuzzard-68F7E71B: G***, kibuzzard-68F7E71B, F.Cu at (157.4, 114.6)
- added kibuzzard-68F7E74E: G***, kibuzzard-68F7E74E, F.Cu at (156.2, 112.5)
- added kibuzzard-68F7E766: G***, kibuzzard-68F7E766, F.Cu at (153.7, 112.2)
- added kibuzzard-68F7E774: G***, kibuzzard-68F7E774, F.Cu at (151.2, 113.5)
- added kibuzzard-68F7E782: G***, kibuzzard-68F7E782, F.Cu at (152.4, 114.1)
- added kibuzzard-68F7E793: G***, kibuzzard-68F7E793, F.Cu at (154.9, 113.8)
- added kibuzzard-690B42CF: G***, kibuzzard-690B42CF, F.Cu at (154.9, 100.2)
- added kibuzzard-690B42EC: G***, kibuzzard-690B42EC, F.Cu at (152.4, 100.2)
- added kibuzzard-690D0FB7: G***, kibuzzard-690D0FB7, F.Cu at (161.3, 112.4)
- added kibuzzard-690D10D3: G***, kibuzzard-690D10D3, F.Cu at (70.7, 110.8)
- added kibuzzard-690D10F1: G***, kibuzzard-690D10F1, F.Cu at (70.7, 104.6)
- added kibuzzard-690D110C: G***, kibuzzard-690D110C, F.Cu at (152.2, 129.3)
- moved D3 0.35 mm to (69.0, 111.2)
- moved R3 0.35 mm to (69.0, 116.2)
Routing:
- net +3.3V: track 260.0 -> 262.6 mm
- net EN M: track 105.3 -> 105.0 mm, vias 0 -> 1
Other:
- board text added: "By Oscar Yosh GRIVELET"
- board text added: "Carte_Driver 2026_V2"
